File: triple-bypass/triple-bypass.sch (KiCad schematic (older format))
At the start: 68 parts, among them CON101 MD-90SM, J101 HDR1X2, J102 JMP-PCB-3POS, U101 THS7374IPWR, U102 LMV358M8G-13

Commit message: First commit
Parts:
- removed 0V1, 5V1, B1, G1, R1, S1, SL1, SN1, SR2, XL1, XR2, YL1, YR2: TP_50, db-smt:TP50, symbol TP_50
- removed C100, C116, C117: 0.1uF/50V, db-smt:0603, symbol C
- removed C101: 220uF/10V, db-smt:SMD-6.6x6.6, symbol CP
- removed C102, C109, C110: 10uF/10V, db-smt:0805, symbol C_0805
- removed C103, C104, C105, C106, C107, C108: 1uF/16V, db-smt:0603, symbol C
- removed C111, C112: 180pF/50V, db-smt:0603, symbol C
- removed C113, C114, C115: 22uF/10V, db-smt:1206_P, symbol CP_1206
- removed CON101: MD-90SM, db-thparts:MD-90SM, symbol MD-90SM
- removed J101: HDR1X2, db-thparts:HDR1X2, symbol HDR1X2
- removed J102: JMP-PCB-3POS, db-smt:JMP-PCB-3POS, symbol JMP-PCB-3POS
- removed R102, R113, R116, R119: 2.20k, db-smt:0603, symbol R
- removed R103, R104, R105, R106: 5.62k, db-smt:0603, symbol R
- removed R107, R108, R109, R110: 1.00k, db-smt:0603, symbol R
- removed R111: 100k, db-smt:0603, symbol R
- removed R112, R114, R115, R117, R118: 75.0, db-smt:0603, symbol R
- removed R120, R127: 6.19k, db-smt:0603, symbol R
- removed R121, R122, R125, R126: 130k, db-smt:0603, symbol R
- removed R123, R124: 120k, db-smt:0603, symbol R
- removed R128, R129: 10.0k, db-smt:0603, symbol R
- removed R130, R131: 240k, db-smt:0603, symbol R
- removed R132, R133: 332, db-smt:0603, symbol R
- removed U101: THS7374IPWR, db-smt:TSSOP-14, symbol THS7374IPWR
- removed U102: LMV358M8G-13, db-smt:TSSOP-8_3.0mm, symbol LMV358M8G-13
- added FD1, FD2, FD3: Fiducial, Fiducial:Fiducial_0.5mm_Dia_1mm_Outer, symbol Mechanical:MountingHole
- added J1: MD-90SM, CUI_MD-90SM, symbol MD-90SM:MD-90SM
- added LOGO1: Logo_Open_Hardware_Small, Symbol:OSHW-Logo2_7.3x6mm_SilkScreen, symbol Graphic:Logo_Open_Hardware_Small
- added P1, P10, P11, P12, P13, P2, P3, P4, P5, P6, P7, P8, P9: TP_50, TestPoint:TestPoint_Pad_1.5x1.5mm, symbol Mechanical:MountingHole_Pad
Connections:
- net labels removed: 32X-Left, 32X-Right, B-In, G-In, PSG, R-In, SCD-Left, SCD-Right, SYNC-TTL, YM-Left, YM-Right
- wire segments 192 -> 51
- no-connect marks 3 -> 1
Other:
- note removed: "0V to 1510mV signal swing, 2 V/V"
- note removed: "0V to 5V signal \nswing on RGB \nfrom Genesis VDP"
- note removed: "0V to 755mV signal swing \nafter voltage divider"
- note removed: "Bypass the Mega Amp by \nDNP'ing the entire audio \nsection. Simply jumper the\naudio L and R signals \ndirectly onto the -ve pads \nof C114 and C113."
- note removed: "CSYNC from Genesis VDP is \nopen collector output assuming \nthe mod has removed the \nGenesis' own 2.2k pull-up from \nthe signal path"
- note removed: "Logic High on bypass disables \nthe internal filters, logic low \nenables them. Use pin jumper \nto force internal filter."
- note removed: "Mega Amp by ACE and Villahed94\nhttps://tinyurl.com/y83uxgvv"
- note removed: "Notes:\n\n-75 ohm pulldowns on Sega CD & 32x \n can be omitted if still present on console\n (required on 32x inputs if fitting a YM2612 \n in a VA0 to VA1.8 Genesis Model 2)\n\n-2.2K pulldown on YM inputs only required\n if fitting a YM2612 in a console with an \n ASIC YM3438.\n\n-R116 = 750 ohm for Model 2 VA2 & VA2.3"
- note removed: "Select video level or\nTTL csync with PCB\nsolder jumper"
- note removed: "Set C111 and C112 to 47pF if you are \na sadist who enjoys harsh trebly sound\n180pF = 3.684KHz LPF\n47pF = 14.109KHz LPF\n27pF = 24.561KHz LPF"

Commit message: Organize and export pdf
Parts:
- J1: symbol MD-90SM:MD-90SM -> triple-bypass-rescue:MD-90SM-MD-90SM
Changed lines of the file:
@@
 	3200 4400 4100 4400
 $Comp
-L MD-90SM:MD-90SM J1
+L triple-bypass-rescue:MD-90SM-MD-90SM J1
 U 1 1 5C1617D3
 P 8000 2800

Commit message: Increase 5V rail width
Parts:
- J1: symbol triple-bypass-rescue:MD-90SM-MD-90SM -> triple-bypass-rescue:MD-90SM
Changed lines of the file:
@@
 	3200 4400 4100 4400
 $Comp
-L triple-bypass-rescue:MD-90SM-MD-90SM J1
+L triple-bypass-rescue:MD-90SM J1
 U 1 1 5C1617D3
 P 8000 2800
-F 0 "J1" H 7850 3500 50  0000 L CNN
-F 1 "MD-90SM" H 7800 2100 50  0000 L CNN
+F 0 "J1" H 8000 3450 50  0000 C BNN
+F 1 "MD-90SM" H 8000 2100 50  0000 C BNN
 F 2 "CUI_MD-90SM" H 8000 2800 50  0001 L BNN
-F 3 "http://www.cui.com/product/resource/digikeypdf/md-sm-series.pdf" H 8000 2800 50  0001 L BNN
+F 3 "https://www.cui.com/product/resource/digikeypdf/md-sm-series.pdf" H 8000 2800 50  0001 L BNN
 F 4 "CP-2290-ND" H 8000 2800 50  0001 L BNN "Digikey"
 F 5 "CONN RCPT FMALE MINI DIN 9P SLDR" H 8000 2800 50  0001 C CNN "Description"
